Commit message: update lrlite urdf

File: urdf/lrlita/robot.urdf (robot description, URDF)
Before this commit: robot arm_v1, 9 links, 8 joints
Joints:
- joint arm_J5: limit lower=-3.14159265 upper=3.14159265 effort=100 velocity=5.0 -> lower=-6.28 upper=6.28 effort=100 velocity=5.0

Commit message: Update robot.urdf

File: urdf/lrlita/robot.urdf (robot description, URDF)
Before this commit: robot arm_v1, 9 links, 8 joints
Joints:
- joint arm_J4: limit lower=-2.0 upper=2.0 effort=100 velocity=5.0 -> lower=-6.28 upper=6.28 effort=100 velocity=5.0

Commit message: Update robot.urdf

File: urdf/lrlita/robot.urdf (robot description, URDF)
Before this commit: robot arm_v1, 9 links, 8 joints
Joints:
- joint arm_J1: limit lower=-3.14159265 upper=3.14159265 effort=100 velocity=5.0 -> lower=-6.28 upper=6.28 effort=100 velocity=5.0
- joint arm_J2: limit lower=-1.57079632 upper=1.57079632 effort=100 velocity=5.0 -> lower=-6.28 upper=6.28 effort=100 velocity=5.0
- joint arm_J3: limit lower=-3.14159265 upper=3.14159265 effort=100 velocity=5.0 -> lower=-6.28 upper=6.28 effort=100 velocity=5.0

Commit message: Connect to rt_control

File: urdf/lrlita/robot.urdf (robot description, URDF)
Before this commit: robot arm_v1, 9 links, 8 joints
Links:
- link arm_L1: geometry visual mesh filename=package://arm_v1/meshes/arm/L1.STL
- link arm_L2: mass 0.136910629397679 -> 0.6; geometry visual mesh filename=package://arm_v1/meshes/arm/L2.STL
- link arm_L3: mass 0.071034581827702 -> 0.10; geometry visual mesh filename=package://arm_v1/meshes/arm/L3.STL
- link arm_L4: mass 0.022184932643385 -> 0.10; geometry visual mesh filename=package://arm_v1/meshes/arm/L4.STL
- link arm_L5: mass 0.0873760863924216 -> 0.25; geometry visual mesh filename=package://arm_v1/meshes/arm/L5.STL
- link arm_L6: mass 0.0269583221049951 -> 0.15; geometry visual mesh filename=package://arm_v1/meshes/arm/L6.STL
- link arm_base_link: geometry visual mesh filename=package://arm_v1/meshes/arm/base_link.STL
Joints:
- joint arm_J1: limit lower=-6.28 upper=6.28 effort=100 velocity=5.0 -> lower=-3.14159265 upper=3.14159265 effort=100 velocity=5.0
- joint arm_J2: limit lower=-6.28 upper=6.28 effort=100 velocity=5.0 -> lower=-1.57079632 upper=1.57079632 effort=100 velocity=5.0
- joint arm_J3: limit lower=-6.28 upper=6.28 effort=100 velocity=5.0 -> lower=-3.14159265 upper=3.14159265 effort=100 velocity=5.0
- joint arm_J4: limit lower=-6.28 upper=6.28 effort=100 velocity=5.0 -> lower=-3.92699 upper=0.872664 effort=100 velocity=5.0
- joint arm_J5: limit lower=-6.28 upper=6.28 effort=100 velocity=5.0 -> lower=-3.14159265 upper=3.14159265 effort=100 velocity=5.0

Commit message: debug

File: urdf/lrlita/robot.urdf (robot description, URDF)
Before this commit: robot arm_v1, 9 links, 8 joints
Links:
- link arm_L1: geometry visual mesh filename=meshes/visual/L1.STL
- link arm_L2: geometry visual mesh filename=meshes/visual/L2.STL
- link arm_L3: geometry visual mesh filename=meshes/visual/L3.STL
- link arm_L4: geometry visual mesh filename=meshes/visual/L4.STL
- link arm_L5: geometry visual mesh filename=meshes/visual/L5.STL
- link arm_L6: geometry visual mesh filename=meshes/visual/L6.STL
- link arm_base_link: geometry visual mesh filename=meshes/visual/base_link.STL
