Commit message: update use sdk,support spark2

File: urdf/spark/robot.urdf (robot description, URDF)
Before this commit: robot spark2, 9 links, 8 joints
Links:
- link arm_L1: geometry visual mesh filename=meshes/visual/L1.STL
- link arm_L2: geometry visual mesh filename=meshes/visual/L2.STL
- link arm_L3: geometry visual mesh filename=meshes/visual/L3.STL
- link arm_L4: geometry visual mesh filename=meshes/visual/L4.STL
- link arm_L5: geometry visual mesh filename=meshes/visual/L5.STL
- link arm_L6: geometry visual mesh filename=meshes/visual/L6.STL
- link arm_base_link: geometry visual mesh filename=meshes/visual/base_link.STL

File: urdf/spark2/robot.urdf (robot description, URDF)
Before this commit: robot spark2, 9 links, 8 joints
Links:
- removed link dummy_base_link
- link arm_L1: mass 0.0556965417664696 -> 1.0366445476980894; geometry collision mesh filename=meshes/L1.obj scale=0.001 0.001 0.001; visual mesh filename=meshes/L1.obj scale=0.001 0.001 0.001
- link arm_L2: mass 0.6 -> 1.506641024125369; geometry collision mesh filename=meshes/L2.obj scale=0.001 0.001 0.001; visual mesh filename=meshes/L2.obj scale=0.001 0.001 0.001
- link arm_L3: mass 0.10 -> 0.4975236595473459; geometry collision mesh filename=meshes/L3.obj scale=0.001 0.001 0.001; visual mesh filename=meshes/L3.obj scale=0.001 0.001 0.001
- link arm_L4: mass 0.10 -> 0.05610708650016425; geometry collision mesh filename=meshes/L4.obj scale=0.001 0.001 0.001; visual mesh filename=meshes/L4.obj scale=0.001 0.001 0.001
- link arm_L5: mass 0.25 -> 0.7330014758686225; geometry collision mesh filename=meshes/L5.obj scale=0.001 0.001 0.001; visual mesh filename=meshes/L5.obj scale=0.001 0.001 0.001
- link arm_L6: mass 0.15 -> 0.049166120435743116; geometry collision mesh filename=meshes/L6.obj scale=0.001 0.001 0.001; visual mesh filename=meshes/L6.obj scale=0.001 0.001 0.001
- link arm_base_link: mass 0.294119348658744 -> 0.8810661689456585; geometry collision mesh filename=meshes/base_link.obj scale=0.001 0.001 0.001; visual mesh filename=meshes/base_link.obj scale=0.001 0.001 0.001
Joints:
- removed joint J0
- joint arm_J1: limit lower=-3.14159265 upper=3.14159265 effort=100 velocity=5.0 -> lower=-3.141593 upper=3.141593 effort=100 velocity=100; origin xyz=0.000000000 0.000000000 0.0962      rpy=0.000000000 0.000000000 0.000000000 -> xyz=0 0 0.084000000000000005 rpy=0 0 0
- joint arm_J2: limit lower=-1.57079632 upper=1.57079632 effort=100 velocity=5.0 -> lower=-1.570796 upper=1.570796 effort=100 velocity=100; origin xyz= 0.0965       0.000000000  0.000000000 rpy= -1.57079632  -1.57079632  0.000000000 -> xyz=0.096000000000000002 0 0 rpy=-1.5707963267948966 -1.5707963267948966 0
- joint arm_J3: limit lower=-3.14159265 upper=3.14159265 effort=100 velocity=5.0 -> lower=-3.141593 upper=3.141593 effort=100 velocity=100; origin xyz= 0.3465       0.000000000  0.000000000 rpy= 0.000000000  0.000000000  0.000000000 -> xyz=0.34649999999999997 0 0 rpy=0 0 0
- joint arm_J4: limit lower=-3.92699 upper=0.872664 effort=100 velocity=5.0 -> lower=-0.349066 upper=3.141593 effort=100 velocity=100; origin xyz= 0.15         0.000000000  0.000000000 rpy= 0.000000000  0.000000000  0.000000000 -> xyz=0.14999999999999999 0 0 rpy=0 0 0
- joint arm_J5: limit lower=-3.14159265 upper=3.14159265 effort=100 velocity=5.0 -> lower=-3.141593 upper=3.141593 effort=100 velocity=100; origin xyz= 0.000000000  0.0965      0.000000000 rpy= -1.57079632  -1.57079632  0.000000000 -> xyz=0 -0.096000000000000002 0 rpy=1.5707963267948966 -1.5707963267948966 0
- joint arm_J6: limit lower=-6.2831853 upper=6.2831853 effort=100 velocity=5.0 -> lower=-6.2831853 upper=6.2831853 effort=100 velocity=100; origin xyz= 0.000000000  0.185  0.000000000 rpy= -1.57079632  0.000000000  0.000000000 -> xyz=0 -0.20000000000000001 0 rpy=1.5707963267948966 0 0
- joint arm_J7: origin xyz=0.045 0 0 rpy=0 0 0 -> xyz=0 0 0 rpy=0 0 0
