Commit message: update URDF

File: urdf/spark2_v1/robot.urdf (robot description, URDF)
Before this commit: robot spark2, 9 links, 8 joints
Joints:
- joint arm_J7: origin xyz=0.045 0 0 rpy=0 0 0 -> xyz=0 0 0.0146 rpy=0 0 0

File: urdf/spark2_v2_2/robot.urdf (robot description, URDF)
Before this commit: robot spark2, 8 links, 7 joints
Links:
- removed link arm_L1
- removed link arm_L2
- removed link arm_L3
- removed link arm_L4
- removed link arm_L5
- removed link arm_L6
- removed link arm_base_link
- added link L1, mass 0.534905861017287; collision mesh filename=meshes/L1.STL; visual mesh filename=meshes/L1.STL
- added link L2, mass 1.04321954132946; collision mesh filename=meshes/L2.STL; visual mesh filename=meshes/L2.STL
- added link L3, mass 0.604374693422943; collision mesh filename=meshes/L3.STL; visual mesh filename=meshes/L3.STL
- added link L4, mass 0.0680910386855528; collision mesh filename=meshes/L4.STL; visual mesh filename=meshes/L4.STL
- added link L5, mass 0.666007703225141; collision mesh filename=meshes/L5.STL; visual mesh filename=meshes/L5.STL
- added link L6, mass 0.0600936238717863; collision mesh filename=meshes/L6.STL; visual mesh filename=meshes/L6.STL
- added link base_link, mass 0.415365145484454; collision mesh filename=meshes/base_link.STL; visual mesh filename=meshes/base_link.STL
Joints:
- removed joint arm_J1
- removed joint arm_J2
- removed joint arm_J3
- removed joint arm_J4
- removed joint arm_J5
- removed joint arm_J6
- removed joint arm_J7
- added joint J1: type revolute, parent base_link, child L1, origin xyz=0 0 0.0982000000000019 rpy=0 0 0, axis 0 0 1, limit lower=-3.1416 upper=3.1416 effort=0 velocity=0
- added joint J2: type revolute, parent L1, child L2, origin xyz=0.096 0 0 rpy=-1.5708 -1.5708 0, axis 0 0 1, limit lower=-1.5708 upper=1.5708 effort=0 velocity=0
- added joint J3: type revolute, parent L2, child L3, origin xyz=0.3465 0 0 rpy=0 0 0, axis 0 0 1, limit lower=-3.1416 upper=3.1416 effort=0 velocity=0
- added joint J4: type revolute, parent L3, child L4, origin xyz=0.15 0 0 rpy=0 0 0, axis 0 0 1, limit lower=-0.1745 upper=3.1416 effort=0 velocity=0
- added joint J5: type revolute, parent L4, child L5, origin xyz=0 -0.09572 0 rpy=1.5708 -1.5708 0, axis 0 0 1, limit lower=-3.1416 upper=3.1416 effort=0 velocity=0
- added joint J6: type revolute, parent L5, child L6, origin xyz=0 -0.1189 0 rpy=1.5708 0 0, axis 0 0 1, limit lower=-6.2832 upper=6.2832 effort=0 velocity=0
- added joint J7: type fixed, parent L6, child arm_end_effector, origin xyz=0 0 0.0146 rpy=0 0 0
