Commit message: Default spark2_v2_2;modify urdf switch in phone

File: urdf/spark2_v2/robot.urdf (robot description, URDF)
Before this commit: robot spark2, 8 links, 7 joints
Links:
- link arm_L1: geometry collision mesh filename=meshes/L1.stl scale=0.001 0.001 0.001; visual mesh filename=meshes/L1.obj scale=0.001 0.001 0.001
- link arm_L2: geometry collision mesh filename=meshes/L2.stl scale=0.001 0.001 0.001; visual mesh filename=meshes/L2.obj scale=0.001 0.001 0.001
- link arm_L3: geometry collision mesh filename=meshes/L3.stl scale=0.001 0.001 0.001; visual mesh filename=meshes/L3.obj scale=0.001 0.001 0.001
- link arm_L4: geometry collision mesh filename=meshes/L4.stl scale=0.001 0.001 0.001; visual mesh filename=meshes/L4.obj scale=0.001 0.001 0.001
- link arm_L5: geometry collision mesh filename=meshes/L5.stl scale=0.001 0.001 0.001; visual mesh filename=meshes/L5.obj scale=0.001 0.001 0.001
- link arm_L6: geometry collision mesh filename=meshes/L6.stl scale=0.001 0.001 0.001; visual mesh filename=meshes/L6.obj scale=0.001 0.001 0.001
- link arm_base_link: geometry collision mesh filename=meshes/base_link.stl scale=0.001 0.001 0.001; visual mesh filename=meshes/base_link.obj scale=0.001 0.001 0.001

Commit message: add log for urdf slow

File: urdf/spark2_v2/robot.urdf (robot description, URDF)
Before this commit: robot spark2, 8 links, 7 joints
Links:
- link arm_L1: geometry collision mesh filename=meshes/L1.obj scale=0.001 0.001 0.001; visual mesh filename=meshes/L1.obj scale=0.001 0.001 0.001
- link arm_L2: geometry collision mesh filename=meshes/L2.obj scale=0.001 0.001 0.001; visual mesh filename=meshes/L2.obj scale=0.001 0.001 0.001
- link arm_L3: geometry collision mesh filename=meshes/L3.obj scale=0.001 0.001 0.001; visual mesh filename=meshes/L3.obj scale=0.001 0.001 0.001
- link arm_L4: geometry collision mesh filename=meshes/L4.obj scale=0.001 0.001 0.001; visual mesh filename=meshes/L4.obj scale=0.001 0.001 0.001
- link arm_L5: geometry collision mesh filename=meshes/L5.obj scale=0.001 0.001 0.001; visual mesh filename=meshes/L5.obj scale=0.001 0.001 0.001
- link arm_L6: geometry collision mesh filename=meshes/L6.obj scale=0.001 0.001 0.001; visual mesh filename=meshes/L6.obj scale=0.001 0.001 0.001
- link arm_base_link: geometry collision mesh filename=meshes/base_link.obj scale=0.001 0.001 0.001; visual mesh filename=meshes/base_link.obj scale=0.001 0.001 0.001
