Commit message: update gripper

File: urdf/spark2_v2_2_with_gripper/robot.urdf (robot description, URDF)
Before this commit: robot spark2_v2_2, 11 links, 10 joints
Links:
- link gripper_L1: mass 0.0622508734002078 -> 0.068045
- link gripper_L2: mass 0.0622502347047371 -> 0
- link gripper_base_link: mass 0.180107205767477 -> 0.139307939402755
Joints:
- joint gripper_J1: limit lower=-0.03 upper=0.01 effort=10 velocity=10 -> lower=-0.0477 upper=0 effort=5 velocity=10; origin xyz=0.031745 0 0.18389 rpy=1.5708 0 -1.5708 -> xyz=0.047697 0 0.16189 rpy=1.5708 0 -1.5708
- joint gripper_J1_1: limit lower=-0.01 upper=0.03 effort=10 velocity=10 -> lower=0 upper=0.0477 effort=5 velocity=10; origin xyz=-0.031745 0 0.18188 rpy=1.5708 0 1.5708 -> xyz=-0.047697 0 0.16188 rpy=1.5708 0 1.5708
