Commit message: update URDF

File: urdf/spark2_v2_2/robot.urdf (robot description, URDF)
Before this commit: robot spark2_v2_2, 8 links, 7 joints
Links:
- link L1: geometry collision mesh filename=meshes/L1,stl; visual mesh filename=meshes/L1,stl
- link L2: geometry collision mesh filename=meshes/L2,stl; visual mesh filename=meshes/L2,stl
- link L3: geometry collision mesh filename=meshes/L3,stl; visual mesh filename=meshes/L3,stl
- link L4: geometry collision mesh filename=meshes/L4,stl; visual mesh filename=meshes/L4,stl
- link L5: geometry collision mesh filename=meshes/L5,stl; visual mesh filename=meshes/L5,stl
- link L6: geometry collision mesh filename=meshes/L6,stl; visual mesh filename=meshes/L6,stl
- link base_link: geometry collision mesh filename=meshes/base_link,stl; visual mesh filename=meshes/base_link,stl

Commit message: update URDF

File: urdf/spark2_v2_2/robot.urdf (robot description, URDF)
Before this commit: robot spark2_v2_2, 8 links, 7 joints
Links:
- link L1: geometry collision mesh filename=meshes/L1.stl; visual mesh filename=meshes/L1.stl
- link L2: geometry collision mesh filename=meshes/L2.stl; visual mesh filename=meshes/L2.stl
- link L3: geometry collision mesh filename=meshes/L3.stl; visual mesh filename=meshes/L3.stl
- link L4: geometry collision mesh filename=meshes/L4.stl; visual mesh filename=meshes/L4.stl
- link L5: geometry collision mesh filename=meshes/L5.stl; visual mesh filename=meshes/L5.stl
- link L6: geometry collision mesh filename=meshes/L6.stl; visual mesh filename=meshes/L6.stl
- link base_link: geometry collision mesh filename=meshes/base_link.stl; visual mesh filename=meshes/base_link.stl

Commit message: add spark2_v2_2 obj mesh

File: urdf/spark2_v2_2/robot.urdf (robot description, URDF)
Before this commit: robot spark2_v2_2, 8 links, 7 joints
Links:
- link L1: geometry collision mesh filename=meshes/L1.obj; visual mesh filename=meshes/L1.obj
- link L2: geometry collision mesh filename=meshes/L2.obj; visual mesh filename=meshes/L2.obj
- link L3: geometry collision mesh filename=meshes/L3.obj; visual mesh filename=meshes/L3.obj
- link L4: geometry collision mesh filename=meshes/L4.obj; visual mesh filename=meshes/L4.obj
- link L5: geometry collision mesh filename=meshes/L5.obj; visual mesh filename=meshes/L5.obj
- link L6: geometry collision mesh filename=meshes/L6.obj; visual mesh filename=meshes/L6.obj
- link base_link: geometry collision mesh filename=meshes/base_link.obj; visual mesh filename=meshes/base_link.obj

Commit message: Remove the spark2_v2_2's flange

File: urdf/spark2_v2_2/robot.urdf (robot description, URDF)
Before this commit: robot spark2_v2_2, 8 links, 7 joints
Joints:
- joint J7: origin xyz=0 0 0.0146 rpy=0 0 0 -> xyz=0 0 0 rpy=0 0 0
